File: pcb/pcb.kicad_pcb (KiCad board)
At the start: 2 copper layers, 234.6 x 93.6 mm, 85 parts, among them SW1 SW_PUSH, SW10 SW_PUSH, SW11 SW_PUSH, SW12 SW_PUSH, SW13 SW_PUSH, SW14 SW_PUSH, SW15 SW_PUSH, SW16 SW_PUSH, SW17 SW_PUSH, SW18 SW_PUSH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

Commit message: Add files via upload
Routing:
- net (no net): track 183.5 -> 1.16 mm
- net +BATT: track 0.00 -> 97.4 mm
- net -BATT: track 0.00 -> 84.9 mm
Other:
- net class Default removed
- net class Power removed
